File: usb2RF.sch (KiCad schematic (older format))
At the start: 38 parts, among them J1 USB_B_Micro, J2 SMA, J3 ARM 10Pin, U1 nRF24L01P, U2 XC6206P332MR, U3 USBLC6-2SC6, U4 STM32L432KBU6, Y1 16MHz

Commit message: [reLayout] [Router] Partially [FrontSilk]ZoomIn
Signed-off-by: EasonLiang <liangyx25@163.com>
Parts:
- J1: footprint Connector_USB:USB_Micro-B_Molex-105017-0001 -> Connector_USB:USB_Mini-B_Lumberg_2486_01_Horizontal; symbol Connector:USB_B_Micro -> usb2RF-rescue:USB_B_Micro-Connector
- J2: symbol Connector:Conn_Coaxial -> usb2RF-rescue:Conn_Coaxial-Connector
Changed lines of the file:
@@
 	8300 5150 8300 5100
 $Comp
-L Connector:USB_B_Micro J1
+L usb2RF-rescue:USB_B_Micro-Connector J1
 U 1 1 60E915C1
 P 4050 1600
 F 0 "J1" H 4107 2067 50  0000 C CNN
 F 1 "USB_B_Micro" H 4107 1976 50  0000 C CNN
-F 2 "Connector_USB:USB_Micro-B_Molex-105017-0001" H 4200 1550 50  0001 C CNN
+F 2 "Connector_USB:USB_Mini-B_Lumberg_2486_01_Horizontal" H 4200 1550 50  0001 C CNN
 F 3 "~" H 4200 1550 50  0001 C CNN
 	1    4050 1600
@@
 $EndComp
 $Comp
-L Connector:Conn_Coaxial J2
+L usb2RF-rescue:Conn_Coaxial-Connector J2
 U 1 1 60FDCC4D
 P 6750 3900
@@
 	7700 4850 10600 4850
 $Comp
-L power:+5V #PWR?
+L power:+5V #PWR0101
 U 1 1 60FAB9E9
 P 5200 1500
-F 0 "#PWR?" H 5200 1350 50  0001 C CNN
+F 0 "#PWR0101" H 5200 1350 50  0001 C CNN
 F 1 "+5V" H 5300 1600 50  0000 C CNN
 F 2 "" H 5200 1500 50  0001 C CNN

Commit message: [library List] both [PCB] update [schematic] update footprint
Signed-off-by: EasonLiang <liang_yongxin@apple.com>
Parts:
- J1: footprint Connector_USB:USB_Mini-B_Lumberg_2486_01_Horizontal -> pcbEsLib:USB-Micro; symbol usb2RF-rescue:USB_B_Micro-Connector -> schEsLib:USB_Micro
- J2: footprint Connector_Coaxial:SMA_Samtec_SMA-J-P-X-ST-EM1_EdgeMount -> pcbEsLib:SMA_EdgeMount; symbol usb2RF-rescue:Conn_Coaxial-Connector -> Connector:Conn_Coaxial
Changed lines of the file:
@@
 	8300 5150 8300 5100
 $Comp
-L usb2RF-rescue:USB_B_Micro-Connector J1
+L schEsLib:USB_Micro J1
 U 1 1 60E915C1
 P 4050 1600
 F 0 "J1" H 4107 2067 50  0000 C CNN
 F 1 "USB_B_Micro" H 4107 1976 50  0000 C CNN
-F 2 "Connector_USB:USB_Mini-B_Lumberg_2486_01_Horizontal" H 4200 1550 50  0001 C CNN
+F 2 "pcbEsLib:USB-Micro" H 4200 1550 50  0001 C CNN
 F 3 "~" H 4200 1550 50  0001 C CNN
 	1    4050 1600
@@
 $EndComp
 $Comp
-L usb2RF-rescue:Conn_Coaxial-Connector J2
+L Connector:Conn_Coaxial J2
 U 1 1 60FDCC4D
 P 6750 3900
 F 0 "J2" H 6850 3875 50  0000 L CNN
 F 1 "SMA" H 6850 3784 50  0000 L CNN
-F 2 "Connector_Coaxial:SMA_Samtec_SMA-J-P-X-ST-EM1_EdgeMount" H 6750 3900 50  0001 C CNN
+F 2 "pcbEsLib:SMA_EdgeMount" H 6750 3900 50  0001 C CNN
 F 3 " ~" H 6750 3900 50  0001 C CNN
 	1    6750 3900

Commit message: [footprint] update for decoupling capacitor for NRF24L01
Signed-off-by: EasonLiang <liangyx25@163.com>
Parts:
- C1: footprint Capacitor_SMD:C_0402_1005Metric -> Capacitor_SMD:C_0603_1608Metric
Changed lines of the file:
@@
 F 0 "C1" H 1165 3396 50  0000 L CNN
 F 1 "10uF" H 1165 3305 50  0000 L CNN
-F 2 "Capacitor_SMD:C_0402_1005Metric" H 1088 3200 50  0001 C CNN
+F 2 "Capacitor_SMD:C_0603_1608Metric" H 1088 3200 50  0001 C CNN
 F 3 "~" H 1050 3350 50  0001 C CNN
 	1    1050 3350
